File: hardware/ControlBoard/ControlBoard.kicad_pcb (KiCad board)
At the start: 2 copper layers, 50.4 x 69.6 mm, 27 parts, among them J1 Power, J2 LCD, J3 SSR, SW1 BUT_A, SW2 BUT_B, SW3 Rotary_Encoder_Switch, U1 DS18B20, U2 LM7805_TO220

Commit message: PCB cleanup
Parts:
- removed G***: LOGO, ControlBoard:Untitled
- removed the REF** at (133.1, 60.2)
